File: workspace/systemMonitorLab/hardware/NodoAmbienteSMN/NodoV2/PcbSistemaAmbienteLab_shield_base_2.kicad_pcb (KiCad board)
At the start: 2 copper layers, 57 x 78 mm, 19 parts, among them J1 Molex_MainBoard_DHT22, J2 Molex_MainBoard_BMP280, J3 Molex_MainBoard_Led_Status, J4 DC 5V, Q1 NPN, Q2 NPN, Q3 NPN, U1 NodeMcuEsp8266

Commit message: Agrego los negativos para su impresion
Parts:
- added ?: , , F.Cu at (125.3, 110.2)
- added ?: , , F.Cu at (154.8, 81.0)
Changed lines of the file:
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@@
+	(footprint ""
+		(layer "F.Cu")
+		(at 125.295 110.21)
+		(property "Reference" ""
+			(at 0 0 0)
+			(layer "F.SilkS")
+			(effects
+				(font
+					(size 1.27 1.27)
+					(thickness 0.15)
+				)
+			)
+		)
+		(property "Value" ""
+			(at 0 0 0)
+			(layer "F.Fab")
+			(effects
+				(font
+					(size 1.27 1.27)
+					(thickness 0.15)
+				)
+			)
+		)
+		(property "Datasheet" ""
+			(at 0 0 0)
+			(layer "F.Fab")
+			(hide yes)
+			(effects
+				(font
+					(size 1.27 1.27)
+					(thickness 0.15)
+				)
+			)
+		)
+		(property "Description" ""
+			(at 0 0 0)
+			(layer "F.Fab")
+			(hide yes)
+			(effects
+				(font
+					(size 1.27 1.27)
+					(thickness 0.15)
+				)
+			)
+		)
+		(pad "" thru_hole circle
+			(at 0 0 270)
+			(size 3 3)
+			(drill 1)
+			(layers "*.Cu" "*.Mask")
+			(remove_unused_layers no)
+			(pinfunction "RV")
+			(pintype "bidirectional+no_connect")
+		)
+		(embedded_fonts no)
+	)
 	(footprint ""
 		(layer "F.Cu")
@@
 		)
 	)
+	(footprint ""
+		(layer "F.Cu")
+		(at 154.775 81.01)
+		(property "Reference" ""
+			(at 0 0 0)
+			(layer "F.SilkS")
+			(effects
+				(font
+					(size 1.27 1.27)
+					(thickness 0.15)
+				)
+			)
+		)
+		(property "Value" ""
+			(at 0 0 0)
+			(layer "F.Fab")
+			(effects
+				(font
+					(size 1.27 1.27)
+					(thickness 0.15)
+				)
+			)
+		)
+		(property "Datasheet" ""
+			(at 0 0 0)
+			(layer "F.Fab")
+			(hide yes)
+			(effects
+				(font
+					(size 1.27 1.27)
+					(thickness 0.15)
+				)
+			)
+		)
+		(property "Description" ""
+			(at 0 0 0)
+			(layer "F.Fab")
+			(hide yes)
+			(effects
+				(font
+					(size 1.27 1.27)
+					(thickness 0.15)
+				)
+			)
+		)
+		(pad "" thru_hole circle
+			(at 0 0 270)
+			(size 3 3)
+			(drill 1)
+			(layers "*.Cu" "*.Mask")
+			(remove_unused_layers no)
+			(pinfunction "RV")
+			(pintype "bidirectional+no_connect")
+		)
+		(embedded_fonts no)
+	)
 	(footprint "Connector_PinHeader_2.54mm:PinHeader_1x04_P2.54mm_Horizontal"

Commit message: Se mejora el plano de masa del PCB
Parts:
- U1: footprint Module_commercial:ESP8266_v3 -> Library:ESP8266_v3
Changed lines of the file:
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@@
 		(grid_origin 116.825 131.21)
 		(pcbplotparams
-			(layerselection 0x00000000_00000000_55555555_5755f5ff)
+			(layerselection 0x00000000_00000000_55555555_55555554)
 			(plot_on_all_layers_selection 0x00000000_00000000_00000000_00000000)
 			(disableapertmacros no)
@@
 			(dxfimperialunits yes)
 			(dxfusepcbnewfont yes)
-			(psnegative no)
+			(psnegative yes)
 			(psa4output no)
 			(plot_black_and_white yes)
-			(plotinvisibletext no)
 			(sketchpadsonfab no)
 			(plotpadnumbers no)
@@
 			(crossoutdnponfab yes)
 			(subtractmaskfromsilk no)
-			(outputformat 1)
+			(outputformat 4)
 			(mirror no)
-			(drillshape 1)
+			(drillshape 0)
 			(scaleselection 1)
-			(outputdirectory "")
+			(outputdirectory "./")
 		)
 	)
@@
 		(embedded_fonts no)
 	)
-	(footprint "Module_commercial:ESP8266_v3"
+	(footprint "Library:ESP8266_v3"
 		(layer "F.Cu")
 		(at 133.25 130.6925)
@@
 			(keep_text_aligned yes)
 		)
-		(gr_text "78.0000 mm"
+		(gr_text "78,0000 mm"
 			(at 189.105 97.96 90)
 			(layer "Dwgs.User")
@@
 			(keep_text_aligned yes)
 		)
-		(gr_text "57.0000 mm"
+		(gr_text "57,0000 mm"
 			(at 143.275 50.77 0)
 			(layer "Dwgs.User")
@@
 			(keep_text_aligned yes)
 		)
-		(gr_text "46.0000 mm"
+		(gr_text "46,0000 mm"
 			(at 143.45 144.21 0)
 			(layer "Dwgs.User")
@@
 			(keep_text_aligned yes)
 		)
-		(gr_text "67.5000 mm"
+		(gr_text "67,5000 mm"
 			(at 105.65 97.86 90)
 			(layer "Dwgs.User")
